Commit message: Replace properties by arguments + colorize links

File: diffbot2_description/urdf/diffbot2.xacro (robot description, xacro)
@@ -2,10 +2,10 @@
 <robot name="diffbot2"
   xmlns:xacro="http://ros.org/wiki/xacro">
-  <!-- Properties -->
-  <xacro:arg name="base_width" default="0.3"/>
-  <xacro:property name="base_length" default="0.4"/>
-  <xacro:property name="base_height" default="0.08"/>
-  <xacro:property name="wheel_radius" default="0.05"/>
-  <xacro:property name="wheel_thickness" default="0.1"/>
+  <!-- Arguments -->
+  <xacro:arg name="base_width" default="0.5"/>
+  <xacro:arg name="base_length" default="0.8"/>
+  <xacro:arg name="base_height" default="0.2"/>
+  <xacro:arg name="wheel_radius" default="0.2"/>
+  <xacro:arg name="wheel_thickness" default="0.1"/>
   <!-- Include macros -->
   <xacro:include filename="$(find diffbot2_description)/urdf/wheel.xacro"/>
@@ -19,20 +19,23 @@
     <visual>
       <geometry>
-        <box size="${base_length} $(arg base_width) ${base_height}"/>
+        <box size="$(arg base_length) $(arg base_width) $(arg base_height)"/>
       </geometry>
+      <material name="white">
+        <color rgba="1 1 1 1"/>
+      </material>
     </visual>
     <collision>
       <origin xyz="0 0 0"/>
       <geometry>
-        <box size="${base_length} $(arg base_width) ${base_height}"/>
+        <box size="$(arg base_length) $(arg base_width) $(arg base_height)"/>
       </geometry>
     </collision>
   </link>
   <!-- Wheels -->
-  <xacro:wheel name="left_wheel" parent="base_link" radius="${wheel_radius}" thickness="${wheel_thickness}">
-    <origin xyz="0 ${$(arg base_width)/2 + wheel_thickness/2} 0" rpy="${-pi/2.} 0 0"/>
+  <xacro:wheel name="left_wheel" parent="base_link" radius="$(arg wheel_radius)" thickness="$(arg wheel_thickness)">
+    <origin xyz="0 ${$(arg base_width)/2 + $(arg wheel_thickness)/2} 0" rpy="${-pi/2.} 0 0"/>
   </xacro:wheel>
-  <xacro:wheel name="right_wheel" parent="base_link" radius="${wheel_radius}" thickness="${wheel_thickness}">
-    <origin xyz="0 ${-$(arg base_width)/2. - wheel_thickness/2.} 0" rpy="${pi/2.} 0 0"/>
+  <xacro:wheel name="right_wheel" parent="base_link" radius="$(arg wheel_radius)" thickness="$(arg wheel_thickness)">
+    <origin xyz="0 ${-$(arg base_width)/2. - $(arg wheel_thickness)/2.} 0" rpy="${pi/2.} 0 0"/>
   </xacro:wheel>
 </robot>

File: diffbot2_description/urdf/wheel.xacro (robot description, xacro)
@@ -12,11 +12,14 @@
         <origin xyz="0 0 0" rpy="0 0 0"/>
         <geometry>
-          <cylinder radius="${wheel_radius}" length="${thickness}"/>
+          <cylinder radius="${radius}" length="${thickness}"/>
         </geometry>
+        <material name="black">
+          <color rgba="0 0 0 1"/>
+        </material>
       </visual>
       <collision>
         <origin xyz="0 0 0" rpy="0 0 0"/>
         <geometry>
-          <cylinder radius="${wheel_radius}" length="${thickness}"/>
+          <cylinder radius="${radius}" length="${thickness}"/>
         </geometry>
       </collision>

Commit message: Fix diffbot2 description
Signed-off-by: Caio Amaral <caioaamaral@gmail.com>

File: diffbot2_description/urdf/diffbot2.xacro (robot description, xacro)
@@ -34,5 +34,5 @@
   <!-- Wheels -->
   <xacro:wheel name="left_wheel" parent="base_link" radius="$(arg wheel_radius)" thickness="$(arg wheel_thickness)">
-    <origin xyz="0 ${$(arg base_width)/2 + $(arg wheel_thickness)/2} 0" rpy="${-pi/2.} 0 0"/>
+    <origin xyz="0 ${$(arg base_width)/2 + $(arg wheel_thickness)/2} 0" rpy="${pi/2.} 0 0"/>
   </xacro:wheel>
   <xacro:wheel name="right_wheel" parent="base_link" radius="$(arg wheel_radius)" thickness="$(arg wheel_thickness)">
@@ -46,5 +46,6 @@
       <right_joint>right_wheel_joint</right_joint>
       <wheel_separation>$(arg base_width)</wheel_separation>
-      <wheel_radius>$(arg base_width)</wheel_radius>
+      <wheel_radius>$(arg wheel_radius)</wheel_radius>
+      <tf_topic>tf</tf_topic>
     </plugin>
   </gazebo>
